Commit message: model update

File: models/hhfc/urdf/hhfc.urdf (robot description, URDF)
Before this commit: robot urdf-20250211, 15 links, 14 joints
Links:
- link Larm_shoulder_p: mass 0.8019 -> 0.9
- link Lleg_ankle_p: mass 0.15381 -> 0.24
- link Lleg_ankle_r: mass 0.87283 -> 0.88; geometry collision mesh filename=../meshes/whole_foot.stl; visual mesh filename=../meshes/whole_foot_visual.stl
- link Lleg_hip_p: mass 0.79889 -> 0.8
- link Lleg_hip_r: mass 2.2937 -> 2.4; geometry visual mesh filename=../meshes/Lleg_hip_r.STL
- link Lleg_hip_y: mass 4.5531 -> 4.7
- link Lleg_knee: mass 4.1746 -> 4.4; geometry visual mesh filename=../meshes/Lleg_knee.STL
- link Rarm_shoulder_p: mass 0.80628 -> 0.9
- link Rleg_ankle_p: mass 0.15381 -> 0.24
- link Rleg_ankle_r: mass 0.87283 -> 0.88; geometry collision mesh filename=../meshes/whole_foot.stl; visual mesh filename=../meshes/whole_foot_visual.stl
- link Rleg_hip_p: mass 0.79889 -> 0.8
- link Rleg_hip_r: mass 2.2802 -> 2.4; geometry visual mesh filename=../meshes/Rleg_hip_r.STL
- link Rleg_hip_y: mass 4.5154 -> 4.7
- link Rleg_knee: mass 4.1724 -> 4.4; geometry visual mesh filename=../meshes/Rleg_knee.STL
- link base_thorax: mass 18.114 -> 20
Joints:
- joint Larm_shoulder_p_joint: limit lower=-3.1416 upper=3.1416 effort=100 velocity=10 -> lower=-3.1416 upper=3.1416 effort=100 velocity=5000; type revolute -> fixed
- joint Lleg_ankle_p_joint: limit lower=-0.6108 upper=0.6108 effort=100 velocity=10 -> lower=-0.6981317007977318 upper=0.6981317007977318 effort=100 velocity=5000
- joint Lleg_ankle_r_joint: limit lower=-0.08727 upper=0.08727 effort=100 velocity=10 -> lower=-0.3490658503988659 upper=0.3490658503988659 effort=100 velocity=5000
- joint Lleg_hip_p_joint: limit lower=-1.5708 upper=3.1416 effort=100 velocity=10 -> lower=-1.5708 upper=3.1416 effort=250 velocity=5000
- joint Lleg_hip_r_joint: limit lower=-0.12217 upper=0.52359 effort=100 velocity=10 -> lower=-0.12217 upper=0.52359 effort=100 velocity=5000
- joint Lleg_hip_y_joint: limit lower=-1.0472 upper=1.2217 effort=100 velocity=10 -> lower=-1.0472 upper=1.2217 effort=100 velocity=5000
- joint Lleg_knee_joint: limit lower=-1.5708 upper=0 effort=100 velocity=10 -> lower=-1.5708 upper=0 effort=250 velocity=5000
- joint Rarm_shoulder_p_joint: limit lower=-3.1416 upper=3.1416 effort=100 velocity=10 -> lower=-3.1416 upper=3.1416 effort=100 velocity=5000; type revolute -> fixed
- joint Rleg_ankle_p_joint: limit lower=-0.6108 upper=0.6108 effort=100 velocity=10 -> lower=-0.6981317007977318 upper=0.6981317007977318 effort=100 velocity=5000
- joint Rleg_ankle_r_joint: limit lower=-0.08727 upper=0.08727 effort=100 velocity=10 -> lower=-0.3490658503988659 upper=0.3490658503988659 effort=100 velocity=5000
- joint Rleg_hip_p_joint: limit lower=-1.5708 upper=3.1416 effort=100 velocity=10 -> lower=-1.5708 upper=3.1416 effort=250 velocity=5000
- joint Rleg_hip_r_joint: limit lower=-0.52359 upper=0.12217 effort=100 velocity=10 -> lower=-0.52359 upper=0.12217 effort=100 velocity=5000
- joint Rleg_hip_y_joint: limit lower=-1.2217 upper=1.0472 effort=100 velocity=10 -> lower=-1.2217 upper=1.0472 effort=100 velocity=5000
- joint Rleg_knee_joint: limit lower=-1.5708 upper=0 effort=100 velocity=10 -> lower=-1.5708 upper=0 effort=250 velocity=5000
