Commit message: updat3

File: models/efc/urdf/efc.urdf (robot description, URDF)
Before this commit: robot sr02h_v1, 25 links, 24 joints
Links:
- link left_ankle_pitch_link: mass 0.0822317248177105 -> 0.2
- link right_ankle_pitch_link: mass 0.0830607206768232 -> 0.2
Joints:
- joint head_joint: type fixed -> revolute
- joint left_elbow_pitch_joint: type fixed -> revolute
- joint left_elbow_yaw_joint: type fixed -> revolute
- joint left_shoulder_pitch_joint: origin xyz=0 0.1665 0.2571 rpy=0 -0.060291 0 -> xyz=0 0.1665 0.2571 rpy=0 0.0 0; type fixed -> revolute
- joint left_shoulder_roll_joint: type fixed -> revolute
- joint left_shoulder_yaw_joint: type fixed -> revolute
- joint right_elbow_pitch_joint: type fixed -> revolute
- joint right_elbow_yaw_joint: type fixed -> revolute
- joint right_shoulder_pitch_joint: origin xyz=0 -0.1665 0.2571 rpy=0 -0.060291 0 -> xyz=0 -0.1665 0.2571 rpy=0 0.0 0; type fixed -> revolute
- joint right_shoulder_roll_joint: type fixed -> revolute
- joint right_shoulder_yaw_joint: type fixed -> revolute
- joint waist_joint: type fixed -> revolute

File: models/efc/urdf/efc_12dof_fake_lim.urdf (robot description, URDF)
Before this commit: robot sr02h_v1, 25 links, 24 joints
Links:
- link left_ankle_pitch_link: mass 0.0822317248177105 -> 0.2
- link right_ankle_pitch_link: mass 0.0830607206768232 -> 0.2
Joints:
- joint left_shoulder_pitch_joint: origin xyz=0 0.1665 0.2571 rpy=0 -0.060291 0 -> xyz=0 0.1665 0.2571 rpy=0 0.0 0
- joint right_shoulder_pitch_joint: origin xyz=0 -0.1665 0.2571 rpy=0 -0.060291 0 -> xyz=0 -0.1665 0.2571 rpy=0 0.0 0

Commit message: update

File: models/efc/urdf/efc.urdf (robot description, URDF)
Before this commit: robot sr02h_v1, 25 links, 24 joints
Links:
- added link world; visual box size=0.01 0.01 0.01
- link right_ankle_roll_link: mass 0.511083104121839 -> 0.528201582069976
Joints:
- added joint world_joint: type revolute, parent world, child base_link, origin xyz=0 0 0 rpy=0 0 0
